File: FT981-AudioCOM.kicad_pcb (KiCad board)
At the start: 2 copper layers, 44 parts, among them J3 USB_B, U1 SL2.1A, U2 CM118B, U3 NCP1117-3.3_SOT223

Commit message: final
Parts:
- removed C12, C7: 100nF, Capacitor_SMD:C_0805_2012Metric
- removed C8: 100uF, Capacitor_SMD:CP_Elec_6.3x5.4
- added C24: 100n, Capacitor_SMD:C_0805_2012Metric, F.Cu at (78.4, 90.3)
- added C31: 100n, Capacitor_SMD:C_0805_2012Metric, F.Cu at (80.5, 90.3)
- added H1: MountingHole, MountingHole:MountingHole_3.2mm_M3_Pad_TopOnly, F.Cu at (72.6, 66.0)
- added H2: MountingHole, MountingHole:MountingHole_3.2mm_M3_Pad_TopOnly, F.Cu at (130.6, 66.0)
- added H3: MountingHole, MountingHole:MountingHole_3.2mm_M3_Pad_TopOnly, F.Cu at (72.6, 127.0)
- added H4: MountingHole, MountingHole:MountingHole_3.2mm_M3_Pad_TopOnly, F.Cu at (130.6, 127.0)
- added J1: Mini-DIN-6, MINI_DIN_6:MINI_DIN_6, F.Cu at (129.8, 83.5)
- added J2: USB_A, USB:USB_A_CONN_LCSC, F.Cu at (84.3, 113.3)
- added Y1: 12MHz, Crystal:Crystal_SMD_3225-4Pin_3.2x2.5mm_HandSoldering, F.Cu at (102.6, 87.0)
- C10, C15, C16, C2, C3, C4, C5, C9: moved to B.Cu
- moved U2 89.9 mm to (82.8, 98.0), turned to -90 degrees
- moved C26 82.2 mm to (80.4, 82.4), turned to 180 degrees
- moved C28 81.4 mm to (80.4, 80.3), turned to 180 degrees
- moved C9 77.4 mm to (80.6, 98.5), turned to 90 degrees
- moved C1 76.8 mm to (76.4, 97.4), turned to 90 degrees
- moved C4 75.4 mm to (77.9, 106.7), turned to 90 degrees
- moved C15 74.3 mm to (82.5, 106.7), turned to -90 degrees
- moved C10 73.7 mm to (84.2, 100.5), turned to 180 degrees
- moved C18 73.5 mm to (90.3, 101.0)
- moved C22 73.4 mm to (87.1, 104.0), turned to -90 degrees
- moved C13 73.0 mm to (97.5, 106.2), turned to 90 degrees
- moved C5 72.5 mm to (80.0, 106.7), turned to 90 degrees
- moved C16 71.4 mm to (84.5, 106.7), turned to -90 degrees
- moved C14 71.1 mm to (82.5, 90.3), turned to 90 degrees
- moved C2 69.9 mm to (82.6, 97.4), turned to -90 degrees
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Connections:
- net Net-(D2-I/O1) renamed /DA-
- net Net-(D2-I/O2) renamed /DA+
- net Net-(D3-I/O1) renamed /DB+
- net Net-(D3-I/O2) renamed /DB-
- net Net-(U1-DM2) renamed /DC-
- net Net-(U1-DP2) renamed /DC+
- U2 pad 11: (no net) -> Net-(C31-Pad1)
- U2 pad 12: (no net) -> Net-(C24-Pad1)
Routing:
- net GND: track 0.00 -> 181.0 mm, vias 0 -> 26
- net +5V: track 0.00 -> 96.5 mm, vias 0 -> 3
- net +5P: track 0.00 -> 68.5 mm, vias 0 -> 2
- net +3.3V: track 0.00 -> 61.8 mm
- net +3.3VA: track 0.00 -> 57.4 mm, vias 0 -> 2
- net DAT_OUT: track 0.00 -> 52.5 mm, vias 0 -> 1
- net DAT_IN: track 0.00 -> 45.9 mm, vias 0 -> 1
- net +5VA: track 0.00 -> 40.4 mm, vias 0 -> 2
- net /DA-: track 0.00 -> 27.5 mm
- net /DA+: track 0.00 -> 27.3 mm
- net /DB+: track 0.00 -> 23.1 mm
- net /DB-: track 0.00 -> 21.8 mm
- net /DC-: track 0.00 -> 9.41 mm
- net /DC+: track 0.00 -> 8.85 mm
- net Net-(U1-XOUT): track 0.00 -> 8.32 mm
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- added copper zone on F.Cu, net +5V
- added copper zone on B.Cu, net GND
Other:
- board outline added: 66.5 x 69.1 mm
