File: FT981-AudioCOM.kicad_sch (KiCad schematic)
At the start: 46 parts, among them J5 USB_A, J7 Mini-DIN-6, J8 USB_B, U1 NCP1117-3.3_SOT223, U2 NCP1117-5.0_SOT223, U5 SL2.1A, U6 CM118B, Y1 12MHz

Commit message: add
Parts:
- removed C10: 100nF, Capacitor_SMD:C_0805_2012Metric, symbol Device:C
- removed C6: 10uF, Capacitor_SMD:C_0805_2012Metric, symbol Device:C_Polarized
- removed U2: NCP1117-5.0_SOT223, Package_TO_SOT_SMD:SOT-223-3_TabPin2, symbol Regulator_Linear:NCP1117-5.0_SOT223
- added C48: 10uF, Capacitor_SMD:C_0805_2012Metric, symbol Device:C
- added R1, R2, R4: 0, Resistor_SMD:R_0805_2012Metric, symbol Device:R
Connections:
- net +12V is gone; now on net +5V: C5.1, C9.1, U1.3 (VI)
- net +3.3VA: now also R4.1; no longer U6.36 (AREG36)
- net AVSS: now also C48.2
- net DAT_IN: now also R2.2; no longer J7.1
- net DAT_OUT: now also R1.2; no longer J7.5
- new net: J7.5, R1.1
- new net: J7.1, R2.1
- new net: C48.1, R4.2, U6.36 (AREG36)
Other:
- moved on the sheet: C13, C14, C18, C19, C20, C21, C5, C9, J7, L4, L5, U1

Commit message: final
Parts:
- removed C37, C42: 100nF, Capacitor_SMD:C_0805_2012Metric, symbol Device:C
- removed C38: 100uF, Capacitor_SMD:CP_Elec_6.3x5.4, symbol Device:C_Polarized
- added C24, C31: 100n, Capacitor_SMD:C_0805_2012Metric, symbol Device:C
- added H1, H2, H3, H4: MountingHole, MountingHole:MountingHole_3.2mm_M3_Pad_TopOnly, symbol Mechanical:MountingHole
- J5: footprint Connectors:USB -> USB:USB_A_CONN_LCSC
- J7: footprint Connectors:Mini-DIN6 -> MINI_DIN_6:MINI_DIN_6
- Y1: footprint (none) -> Crystal:Crystal_SMD_3225-4Pin_3.2x2.5mm_HandSoldering; symbol Device:Crystal -> Device:Crystal_GND24
Connections:
- net AVSS: now also Y1.2, Y1.4, C24.2, C31.2
- net at R1.1: now also J7.6; no longer J7.5
- net DB-: now reaches D24.3 (I/O2), J8.2 (D-), U5.9 (DM)
- net DB+: now reaches D24.2 (I/O1), J8.3 (D+), U5.10 (DP)
- net DC+: now reaches U5.6 (DP2), U6.43 (USBDP)
- net DC-: now reaches U5.5 (DM2), U6.44 (USBDM)
- net at U5.15 (XOUT): now also Y1.3; no longer Y1.2
- net DA-: now reaches D23.2 (I/O1), J5.2 (D-), U5.7 (DM1)
- net DA+: now reaches D23.3 (I/O2), J5.3 (D+), U5.8 (DP1)
- new net: C31.1, U6.11 (DREG18)
- new net: C24.1, U6.12 (DREG33)
